Commit message: Tune controller params and etc

File: kuka_lbr_iiwa_gazebo/urdf/lbr_iiwa_properties.xacro (robot description, xacro)
@@ -2,5 +2,5 @@
 <robot name="kuka_lbr_iiwa_14_r820" xmlns:xacro="http://ros.org/wiki/xacro">
   <!-- ======== ARG SECTION ========= -->
-	<xacro:property name="reduct" value="100" />
+	<xacro:property name="reduct" value="1" />
 	<!-- CAMERA params -->
 	<xacro:property name="PI" value="3.1415926535" />
