Commit message: Add camera link with coordinate frame same as of OpenCV camera model
- now used as tf parent frame for marker

File: kuka_lbr_iiwa_support/urdf/lbr_iiwa_14_r820_macro.xacro (robot description, xacro)
@@ -56,4 +56,5 @@
     </xacro:link_gen>
     <link name="tool0" />
+    <link name="camera_link" />
     <!-- end of link list -->
     <!-- joint list -->
@@ -113,4 +114,10 @@
       <axis xyz="0 0 0" />
     </joint>
+    <joint name="joint_tool0_camera" type="fixed">
+      <origin xyz="0 0 0" rpy="0 0 1.570795" />
+      <parent link="tool0" />
+      <child link="camera_link" />
+      <axis xyz="0 0 0" />
+    </joint>
     <!-- end of joint list -->
     <!-- ROS base_link to KUKA $ROBROOT coordinate system transform -->

Commit message: Add dynamics parameters for joints

File: kuka_lbr_iiwa_support/urdf/lbr_iiwa_14_r820_macro.xacro (robot description, xacro)
@@ -64,4 +64,5 @@
       <child link="link_1" />
       <axis xyz="0 0 1" />
+      <dynamics damping="1.0" friction="5.0"/>
       <limit lower="-2.9668" upper="2.9668" effort="320" velocity="1.4834" />
     </joint>
@@ -71,4 +72,5 @@
       <child link="link_2" />
       <axis xyz="0 1 0" />
+      <dynamics damping="1.0" friction="5.0"/>
       <limit lower="-2.0942" upper="2.0942" effort="320" velocity="1.4834" />
     </joint>
@@ -78,4 +80,5 @@
       <child link="link_3" />
       <axis xyz="0 0 1" />
+      <dynamics damping="1.0" friction="5.0"/>
       <limit lower="-2.9668" upper="2.9668" effort="176" velocity="1.7452" />
     </joint>
@@ -85,4 +88,5 @@
       <child link="link_4" />
       <axis xyz="0 -1 0" />
+      <dynamics damping="1.0" friction="5.0"/>
       <limit lower="-2.0942" upper="2.0942" effort="176" velocity="1.3089" />
     </joint>
@@ -92,4 +96,5 @@
       <child link="link_5" />
       <axis xyz="0 0 1" />
+      <dynamics damping="1.0" friction="5.0"/>
       <limit lower="-2.9668" upper="2.9668" effort="110" velocity="2.2688" />
     </joint>
@@ -99,4 +104,5 @@
       <child link="link_6" />
       <axis xyz="0 1 0" />
+      <dynamics damping="1.0" friction="5.0"/>
       <limit lower="-2.0942" upper="2.0942" effort="40" velocity="2.356" />
     </joint>
@@ -106,4 +112,5 @@
       <child link="link_7" />
       <axis xyz="0 0 1" />
+      <dynamics damping="1.0" friction="5.0"/>
       <limit lower="-3.0541" upper="3.0541" effort="40" velocity="2.356" />
     </joint>
